File: _autosave-valentine.kicad_sch (KiCad schematic)
At the start: 42 parts, among them J1 Conn_01x04_Socket, J2 Battery, SW1 SW_Push_45deg, U1 STM32G031G8Ux

Commit message: pcb design done ,,design as in where to put what i made a grid
Parts:
- J1: footprint Connector_PinSocket_2.54mm:PinSocket_1x04_P2.54mm_Vertical_SMD_Pin1Right -> Connector_PinSocket_2.54mm:PinSocket_2x02_P2.54mm_Vertical_SMD
Connections:
- net PB5: no longer D6.2 (A), U1.11 (PA5)
- net PB6: no longer D7.2 (A), U1.12 (PA6)
- net PB7: no longer D8.2 (A), U1.13 (PA7)
- new net PA5: D6.2 (A), U1.11 (PA5)
- new net PA6: D7.2 (A), U1.12 (PA6)
- new net PA7: D8.2 (A), U1.13 (PA7)
Changed lines of the file:
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@@
 		)
 	)
-	(label "PB7"
+	(label "PA7"
 		(at 88.9 54.61 0)
 		(effects
@@
 		)
 	)
-	(label "PB7"
+	(label "PA7"
 		(at 201.93 50.8 180)
 		(effects
@@
 		)
 	)
-	(label "PB5"
+	(label "PA5"
 		(at 215.9 38.1 180)
 		(effects
@@
 		)
 	)
-	(label "PB6"
+	(label "PA6"
 		(at 189.23 50.8 180)
 		(effects
@@
 		)
 	)
-	(label "PB5"
+	(label "PA5"
 		(at 88.9 49.53 0)
 		(effects
@@
 		)
 	)
-	(label "PB6"
+	(label "PA6"
 		(at 88.9 52.07 0)
 		(effects
@@
 			)
 		)
-		(property "Footprint" "Connector_PinSocket_2.54mm:PinSocket_1x04_P2.54mm_Vertical_SMD_Pin1Right"
+		(property "Footprint" "Connector_PinSocket_2.54mm:PinSocket_2x02_P2.54mm_Vertical_SMD"
 			(at 86.36 93.98 0)
 			(effects
