File: valentine.kicad_sch (KiCad schematic)
At the start: 42 parts, among them J1 Conn_01x04_Socket, J2 Battery, SW1 SW_Push_45deg, U1 STM32G031G8Ux

Commit message: pcb routing
Parts:
- removed D17: LED_STARTUP, LED_SMD:LED_0603_1608Metric, symbol Device:LED
- removed R1: 1.8K, Resistor_SMD:R_0402_1005Metric, symbol Device:R_45deg
- J1: footprint Connector_PinSocket_2.54mm:PinSocket_1x04_P2.54mm_Vertical_SMD_Pin1Right -> Connector_PinSocket_1.27mm:PinSocket_2x02_P1.27mm_Vertical_SMD
Connections:
- net PB5: no longer D6.2 (A), U1.11 (PA5)
- net PB6: no longer D7.2 (A), U1.12 (PA6)
- net PB7: no longer D8.2 (A), U1.13 (PA7)
- net PA8: no longer names the net of U1.16 (PA8)
- new net PA5: D6.2 (A), U1.11 (PA5)
- new net PA6: D7.2 (A), U1.12 (PA6)
- new net PA7: D8.2 (A), U1.13 (PA7)
Changed lines of the file:
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@@
 		)
 	)
-	(label "PB7"
+	(label "PA7"
 		(at 88.9 54.61 0)
 		(effects
@@
 		)
 	)
-	(label "PA8"
-		(at 77.47 57.15 0)
-		(effects
-			(font
-				(size 1.27 1.27)
-			)
-			(justify left bottom)
-		)
-	)
 	(label "PB8"
 		(at 27.94 69.85 180)
@@
 		)
 	)
-	(label "PB7"
+	(label "PA7"
 		(at 201.93 50.8 180)
 		(effects
@@
 		)
 	)
-	(label "PB5"
+	(label "PA5"
 		(at 215.9 38.1 180)
 		(effects
@@
 		)
 	)
-	(label "PB6"
+	(label "PA6"
 		(at 189.23 50.8 180)
 		(effects
@@
 		)
 	)
-	(label "PB5"
+	(label "PA5"
 		(at 88.9 49.53 0)
 		(effects
@@
 		)
 	)
-	(label "PB6"
+	(label "PA6"
 		(at 88.9 52.07 0)
 		(effects
@@
 		)
 	)
-	(label "PA8"
-		(at 190.5 76.2 180)
-		(effects
-			(font
-				(size 1.27 1.27)
-			)
-			(justify right bottom)
-		)
-	)
 	(label "NRST"
 		(at 91.44 88.9 0)
@@
 	)
 	(symbol
-		(lib_id "power:GND")
-		(at 203.2 81.28 0)
-		(unit 1)
-		(exclude_from_sim no)
-		(in_bom yes)
-		(on_board yes)
-		(dnp no)
-		(fields_autoplaced yes)
-		(property "Reference" "#PWR08"
-			(at 203.2 87.63 0)
-			(effects
-				(font
-					(size 1.27 1.27)
-				)
-				(hide yes)
-			)
-		)
-		(property "Value" "GND"
-			(at 203.2 86.36 0)
-			(effects
-				(font
-					(size 1.27 1.27)
-				)
-			)
-		)
-		(property "Footprint" ""
-			(at 203.2 81.28 0)
-			(effects
-				(font
-					(size 1.27 1.27)
-				)
-				(hide yes)
-			)
-		)
-		(property "Datasheet" ""
-			(at 203.2 81.28 0)
-			(effects
-				(font
-					(size 1.27 1.27)
-				)
-				(hide yes)
-			)
-		)
-		(property "Description" "Power symbol creates a global label with name \"GND\" , ground"
-			(at 203.2 81.28 0)
-			(effects
-				(font
-					(size 1.27 1.27)
-				)
-				(hide yes)
-			)
-		)
-		(pin "1"
-		)
-		(instances
-			(project "valentine"
-				(path "/0dba50cb-f61f-4dfb-9895-224e028720eb"
-					(reference "#PWR08")
-					(unit 1)
-				)
-			)
-		)
-	)
-	(symbol
 		(lib_id "Device:LED")
 		(at 245.11 25.4 180)
@@
 	)
 	(symbol
-		(lib_id "Device:R_45deg")
-		(at 200.66 78.74 0)
-		(unit 1)
-		(exclude_from_sim no)
-		(in_bom yes)
-		(on_board yes)
-		(dnp no)
-		(fields_autoplaced yes)
-		(property "Reference" "R1"
-			(at 200.66 71.12 0)
-			(effects
-				(font
-					(size 1.27 1.27)
-				)
-			)
-		)
-		(property "Value" "1.8K"
-			(at 200.66 73.66 0)
-			(effects
-				(font
-					(size 1.27 1.27)
-				)
-			)
-		)
-		(property "Footprint" "Resistor_SMD:R_0402_1005Metric"
-			(at 200.66 80.518 0)
-			(effects
-				(font
-					(size 1.27 1.27)
-				)
-				(hide yes)
-			)
-		)
-		(property "Datasheet" "~"
-			(at 200.66 78.74 0)
-			(effects
-				(font
-					(size 1.27 1.27)
-				)
-				(hide yes)
-			)
-		)
-		(property "Description" "Resistor, rotated by 45°"
-			(at 200.66 78.74 0)
-			(effects
-				(font
-					(size 1.27 1.27)
-				)
-				(hide yes)
-			)
-		)
-		(pin "1"
-		)
-		(pin "2"
-		)
-		(instances
-			(project "valentine"
-				(path "/0dba50cb-f61f-4dfb-9895-224e028720eb"
-					(reference "R1")
-					(unit 1)
-				)
-			)
-		)
-	)
-	(symbol
 		(lib_id "Device:LED")
 		(at 205.74 50.8 180)
@@
 			)
 		)
-		(property "Footprint" "Connector_PinSocket_2.54mm:PinSocket_1x04_P2.54mm_Vertical_SMD_Pin1Right"
+		(property "Footprint" "Connector_PinSocket_1.27mm:PinSocket_2x02_P1.27mm_Vertical_SMD"
 			(at 86.36 93.98 0)
 			(effects
@@
 					(unit 1)
 				)
-			)
-		)
-	)
-	(symbol
-		(lib_id "Device:LED")
-		(at 194.31 76.2 180)
-		(unit 1)
-		(exclude_from_sim no)
-		(in_bom yes)
-		(on_board yes)
-		(dnp no)
-		(property "Reference" "D17"
-			(at 195.8975 68.58 0)
-			(effects
-				(font
-					(size 1.27 1.27)
-				)
-			)
-		)
-		(property "Value" "LED_STARTUP"
-			(at 194.31 80.01 0)
-			(effects
-				(font
-					(size 1.27 1.27)
-				)
-			)
-		)
-		(property "Footprint" "LED_SMD:LED_0603_1608Metric"
-			(at 194.31 76.2 0)
-			(effects
-				(font
-					(size 1.27 1.27)
-				)
-				(hide yes)
-			)
-		)
-		(property "Datasheet" "~"
-			(at 194.31 76.2 0)
-			(effects
-				(font
-					(size 1.27 1.27)
-				)
-				(hide yes)
-			)
-		)
-		(property "Description" "Light emitting diode"
-			(at 194.31 76.2 0)
-			(effects
-				(font
-					(size 1.27 1.27)
-				)
-				(hide yes)
-			)
-		)
-		(property "Sim.Pins" "1=K 2=A"
-			(at 194.31 76.2 0)
-			(effects
-				(font
-					(size 1.27 1.27)
-				)
-				(hide yes)
-			)
-		)
-		(pin "2"
-		)
-		(pin "1"
-		)
-		(instances
-			(project "valentine"
-				(path "/0dba50cb-f61f-4dfb-9895-224e028720eb"
-					(reference "D17")
-					(unit 1)
-				)
